File: AlLock_hw/AlLock.sch (KiCad schematic (older format))
At the start: 135 parts, among them Q2 IRLML6302

Commit message: Uart works
Parts:
- C1, C10, C11, C12, C13, C14, C15, C16, C17, C18, C19, C2, C20, C21, C22, C23, C24, C25, C26, C27, C28, C29, C3, C30, C31, C32, C33, C34, C35, C36, C37, C38, C39, C4, C40, C41, C42, C43, C44, C45, C46, C47, C48, C5, C6, C7, C8, C9: symbol C -> Tittar_kl:C
- D1: symbol D_Shottky -> Tittar_kl:D_Shottky
- DA1: symbol LD1117 -> Power_kl:LD1117
- DA10: symbol NCP3066 -> Power_kl:NCP3066
- DA2: symbol AAT3221 -> Power_kl:AAT3221
- DA3, DA4: symbol IPS6041 -> Power_kl:IPS6041
- DA5: symbol HIN202 -> Interface_kl:HIN202
- DA6: symbol VS1103B -> Audio_kl:VS1103b
- DA7: symbol LP2951 -> Power_kl:LP2951
- DA8: symbol TPA6211 -> Audio_kl:TPA6211
- DD1: symbol STM32F103RC-64 -> st_kl:STM32F103RC-64
- F1, F10, F11, F12, F2, F5, F6, F7, F8, F9: symbol FUSE0R -> Tittar_kl:Fuse0R
- HOLE1, HOLE2, HOLE3, HOLE4: symbol HOLE_METALLED -> pcb_details:HOLE_METALLED
- L1: symbol L -> Tittar_kl:L
- Q2: symbol IRLML6302 -> Transistors_kl:P_3PIN
- R1, R10, R11, R12, R13, R14, R15, R16, R17, R18, R19, R2, R20, R21, R3, R4, R5, R6, R7, R8, R9, R?: symbol R -> Tittar_kl:R
- Rx1, Rx2, Rx3, Rx4: symbol RX4 -> Tittar_kl:RX4
- XL1, XL18, XL2, XL25, XL26, XL27, XL3, XL4, XL5: symbol CONN_2 -> Connectors_kl:CONN_2
- XL10, XL14, XL15, XL16, XL17, XL9: symbol CONN_1 -> Connectors_kl:CONN_1
- XL11: symbol ST_SWD -> Connectors_kl:ST_SWD
- XL12, XL13: symbol CONN_7 -> Connectors_kl:CONN_7
- XL19, XL31: symbol SD_CONNECTOR -> Connectors_kl:SD_CONNECTOR
- XL20, XL21, XL22, XL23, XL24: symbol CONN_4 -> Connectors_kl:CONN_4
- XL28, XL29, XL30, XL6, XL7, XL8: symbol CONN_3 -> Connectors_kl:CONN_3
- XTAL1: symbol CRYSTAL -> Tittar_kl:CRYSTAL
Connections:
- wire segments 478 -> 590
